Commit message: Add files via upload

File: robot_be.urdf (robot description, URDF)
Before this commit: robot robot_be, 4 links, 3 joints
Links:
- removed link outil
- added link corp_3; visual cylinder length=1 radius=0.1
- added link outil_link; visual sphere radius=0.05
Joints:
- added joint outil: type fixed, parent corp_3, child outil_link, origin xyz=0 -1 0 rpy=0 0 0
- joint Rotoide_2: child outil -> corp_3
